Commit message: fix m20 problem

File: M20/urdf/M20.urdf (robot description, URDF)
Before this commit: robot M20, 17 links, 16 joints
Joints:
- joint fl_hipx_joint: limit lower=-0.611 upper=0.436 effort=76.4 velocity=22.4 -> lower=-0.436 upper=0.611 effort=76.4 velocity=22.4
- joint fr_hipx_joint: limit lower=-0.436 upper=0.611 effort=76.4 velocity=22.4 -> lower=-0.611 upper=0.436 effort=76.4 velocity=22.4
- joint hl_hipx_joint: limit lower=-0.611 upper=0.436 effort=76.4 velocity=22.4 -> lower=-0.436 upper=0.611 effort=76.4 velocity=22.4
- joint hr_hipx_joint: limit lower=-0.436 upper=0.611 effort=76.4 velocity=22.4 -> lower=-0.611 upper=0.436 effort=76.4 velocity=22.4

File: M20_Piper/urdf/M20_Piper.urdf (robot description, URDF)
Before this commit: robot M20_Piper, 27 links, 26 joints
Joints:
- joint fl_hipx_joint: limit lower=-0.611 upper=0.436 effort=76.4 velocity=22.4 -> lower=-0.436 upper=0。611 effort=76.4 velocity=22.4
- joint fr_hipx_joint: limit lower=-0.436 upper=0.611 effort=76.4 velocity=22.4 -> lower=-0.611 upper=0.436 effort=76.4 velocity=22.4
- joint hl_hipx_joint: limit lower=-0.611 upper=0.436 effort=76.4 velocity=22.4 -> lower=-0.436 upper=0.611 effort=76.4 velocity=22.4
- joint hr_hipx_joint: limit lower=-0.436 upper=0.611 effort=76.4 velocity=22.4 -> lower=-0.611 upper=0.436 effort=76.4 velocity=22.4

Commit message: feat(robot): 添加传感器框架支持
- 在M20和M20S模型中添加前后摄像头和激光雷达站点定义
- 在URDF文件中添加相应的传感器链接和固定关节配置
- 为X30机器人添加前后上下四个激光雷达的链接定义
- 配置所有传感器的精确位置和方向参数
- 实现毫米到米的单位转换以确保正确的物理模拟
- 添加适当的注释说明传感器框架的来源和规格

File: M20/urdf/M20.urdf (robot description, URDF)
Before this commit: robot M20, 17 links, 16 joints
Links:
- added link front_camera_link
- added link front_lidar_link
- added link rear_camera_link
- added link rear_lidar_link
Joints:
- added joint front_camera_joint: type fixed, parent base_link, child front_camera_link, origin xyz=0.37646 0 0.03738 rpy=0 0 0
- added joint front_lidar_joint: type fixed, parent base_link, child front_lidar_link, origin xyz=0.32028 0 -0.013 rpy=0 0 0
- added joint rear_camera_joint: type fixed, parent base_link, child rear_camera_link, origin xyz=-0.37646 0 0.03738 rpy=0 0 0
- added joint rear_lidar_joint: type fixed, parent base_link, child rear_lidar_link, origin xyz=-0.32028 0 -0.013 rpy=0 0 0

File: M20S/urdf/M20S.urdf (robot description, URDF)
Before this commit: robot M20S, 17 links, 16 joints
Links:
- added link front_camera_link
- added link front_lidar_link
- added link rear_camera_link
- added link rear_lidar_link
Joints:
- added joint front_camera_joint: type fixed, parent base_link, child front_camera_link, origin xyz=0.37646 0 0.03738 rpy=0 0 0
- added joint front_lidar_joint: type fixed, parent base_link, child front_lidar_link, origin xyz=0.32028 0 -0.013 rpy=0 0 0
- added joint rear_camera_joint: type fixed, parent base_link, child rear_camera_link, origin xyz=-0.37646 0 0.03738 rpy=0 0 0
- added joint rear_lidar_joint: type fixed, parent base_link, child rear_lidar_link, origin xyz=-0.32028 0 -0.013 rpy=0 0 0

File: X30/urdf/X30.urdf (robot description, URDF)
Before this commit: robot X30, 17 links, 16 joints
Links:
- added link LIDAR_FRONT_DOWN, mass 1e-5
- added link LIDAR_FRONT_UP, mass 1e-5
- added link LIDAR_REAR_DOWN, mass 1e-5
- added link LIDAR_REAR_UP, mass 1e-5
Joints:
- added joint LIDAR_FRONT_DOWN_joint: type fixed, parent TORSO, child LIDAR_FRONT_DOWN, origin xyz=0.43297 0 -0.05519 rpy=0 0.4363 0
- added joint LIDAR_FRONT_UP_joint: type fixed, parent TORSO, child LIDAR_FRONT_UP, origin xyz=0.44367 0 0.05415 rpy=0 0.4363 0
- added joint LIDAR_REAR_DOWN_joint: type fixed, parent TORSO, child LIDAR_REAR_DOWN, origin xyz=-0.41074 0 -0.05601 rpy=0 -0.8029 0
- added joint LIDAR_REAR_UP_joint: type fixed, parent TORSO, child LIDAR_REAR_UP, origin xyz=-0.46576 0 0.03484 rpy=0 -0.8029 0
